File: Projekt.kicad_pcb (KiCad board)
At the start: 2 copper layers, 93.5 x 60.8 mm, 119 parts, among them J1 Solar, J2 Battery, J3 USB_B_Mini, J4 INTERFACE PORT, J5 FAN, J6 JTAG, J7 PRG, J8 Micro_SD_Card_Det_Hirose_DM3AT, J9 IIC RTC, Q1 CSD19505KCS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

Commit message: Sieht ganz gut aus...
Parts:
- removed J5: FAN, Connector_PinHeader_2.54mm:PinHeader_1x02_P2.54mm_Vertical
- removed J7: PRG, Connector_PinHeader_2.54mm:PinHeader_1x02_P2.54mm_Vertical
- C12, R29, R30: moved to F.Cu
- C21, C22, C24, D10, D11, D12, D13, D14, D9, Q5, Q6, R22, R23, R26, R27, R28, R38, R39, R40, U4: moved to B.Cu
- J4: footprint Connector_PinHeader_2.54mm:PinHeader_1x08_P2.54mm_Vertical -> Connector_PinHeader_1.27mm:PinHeader_2x08_P1.27mm_Vertical_SMD
- JP1: value Copper Bar -> Copper bar
- moved C12 31.1 mm to (154.2, 106.2), turned to 0 degrees
- moved C22 30.0 mm to (137.5, 152.2), turned to -90 degrees
- moved C21 28.0 mm to (127.7, 147.6), turned to 90 degrees
- moved Q6 26.7 mm to (133.0, 135.7)
- moved U4 24.4 mm to (132.6, 150.4), turned to 90 degrees
- moved J4 22.6 mm to (159.3, 118.7), turned to 0 degrees
- moved Q5 20.0 mm to (140.2, 126.2), turned to 90 degrees
- moved D5 19.2 mm to (127.7, 124.7)
- moved R22 17.2 mm to (138.9, 130.0), turned to -90 degrees
- moved C16 15.0 mm to (153.6, 97.9)
- moved R23 14.5 mm to (141.0, 130.0), turned to -90 degrees
- moved R24 14.4 mm to (141.6, 116.9), turned to 90 degrees
- moved C14 12.1 mm to (140.4, 117.2)
- moved C18 11.3 mm to (150.3, 117.2)
- moved C19 10.3 mm to (154.5, 136.3)
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Connections:
- net GPIO12 renamed SD_DAT2
- net GPIO13 renamed SD_DAT3
- net GPIO14 renamed SD_CLK
- net GPIO15 renamed SD_CMD
- net GPIO16 renamed SD_DET_B
- net GPIO27 renamed BCCU
- net GPIO32 renamed DRV_SD
- net GPIO33 renamed DRV_IN
- net GPIO34 renamed ADC_RDY
- net Net-(C21-Pad1) renamed VBUS
- C24 pad 2: GND -> GND2
- C7 pad 2: GND -> GND2
- C8 pad 2: GND -> GND2
- D10 pad 1: GND -> GND2
- D10 pad 2: GPIO25 -> SD_DAT1
- D11 pad 1: GND -> GND2
- D12 pad 1: GND -> GND2
- D13 pad 1: GND -> GND2
- D14 pad 1: GND -> GND2
- D4 pad 2: Net-(D4-Pad2) -> Net-(C8-Pad1)
- D8 pad 2: Net-(D8-Pad2) -> Net-(C7-Pad1)
- D9 pad 1: GPIO26 -> SD_DAT1
- D9 pad 2: GND -> GND2
- F1 pad 1: Net-(D8-Pad2) -> Net-(F1-Pad1)
- F2 pad 1: Net-(D4-Pad2) -> Net-(F2-Pad1)
- J1 pad 1: Net-(D8-Pad2) -> Net-(F1-Pad1)
- J1 pad 2: GND -> GND2
- J2 pad 1: Net-(D4-Pad2) -> Net-(F2-Pad1)
- J2 pad 2: Net-(J2-Pad2) -> GND2
- J3 pad 5: GND -> GND2
- J3 pad 6: GND -> GND2
- J4 pad 1: GND -> +3.3V
- J4 pad 3: SDA -> +12V
- J4 pad 4: SCL -> SDA
- J4 pad 5: GPIO17 -> KEY_LEFT
- J4 pad 6: GPIO18 -> SCL
- J4 pad 7: GPIO19 -> KEY_SELECT
- J4 pad 8: GPIO23 -> KEY_RIGHT
- J8 pad 10: GND -> GND2
- J8 pad 11: GND -> GND2
- J8 pad 6: GND -> GND2
- J8 pad 7: GPIO25 -> SD_DAT1
- J8 pad 8: GPIO26 -> SD_DAT1
- JP1 pad 1: GND -> GND2
- JP1 pad 2: Net-(J2-Pad2) -> GND
- Q6 pad 3: GPIO0 -> PRG
- Q7 pad 1: Net-(Q7-Pad1) -> FAN
- Q7 pad 2: Net-(J5-Pad2) -> FAN_GND
- R24 pad 1: GPIO0 -> PRG
- R25 pad 1: Net-(Q7-Pad1) -> FAN
- R26 pad 2: GPIO26 -> SD_DAT1
- R27 pad 2: GPIO25 -> SD_DAT1
- R29 pad 2: SCL -> SDA
- R30 pad 2: SDA -> SCL
- U5 pad 9: (no net) -> unconnected-(U5-Pad9)
- U6 pad 9: (no net) -> unconnected-(U6-Pad9)
- U8 pad 10: GPIO25 -> SD_DAT1
- U8 pad 11: GPIO26 -> SD_DAT1
- U8 pad 25: GPIO0 -> PRG
- U8 pad 28: GPIO17 -> KEY_RIGHT
- U8 pad 29: unconnected-(U8-Pad29) -> FAN
- U8 pad 30: GPIO18 -> KEY_LEFT
- U8 pad 31: GPIO19 -> KEY_BACK
- U8 pad 37: GPIO23 -> KEY_SELECT
Routing:
- net GND: track 95.3 -> 588.4 mm, vias 0 -> 17
- net +3.3V: track 0.00 -> 250.4 mm, vias 0 -> 21
- net GND2: track 0.00 -> 201.5 mm, vias 0 -> 4
- net SDA: track 0.00 -> 184.6 mm, vias 0 -> 8
- net +12V: track 0.00 -> 170.3 mm, vias 0 -> 11
- net Net-(C12-Pad1): track 0.00 -> 138.2 mm, vias 0 -> 6
- net A2: track 0.00 -> 135.7 mm, vias 0 -> 8
- net SD_DET_B: track 0.00 -> 107.7 mm, vias 0 -> 7
- net Net-(C7-Pad1): track 18.8 -> 121.4 mm, vias 0 -> 7
- net +5V: track 0.00 -> 100.7 mm, vias 0 -> 3
- net BCCU: track 0.00 -> 85.8 mm, vias 0 -> 3
- net Net-(LED1-Pad2): track 0.00 -> 84.7 mm, vias 0 -> 3
- net Net-(D2-Pad1): track 0.00 -> 83.1 mm, vias 0 -> 2
- net Net-(C10-Pad2): track 56.7 -> 127.5 mm, vias 0 -> 1
- net SD_CLK: track 0.00 -> 69.5 mm, vias 0 -> 7
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Other:
- board size 93.5 x 60.8 mm -> 86.8 x 60.8 mm
