File: MPPT_Charger.kicad_pcb (KiCad board)
At the start: 2 copper layers, 86.8 x 60.8 mm, 118 parts, among them J1 Solar, J2 Battery, J3 USB_B_Mini, J4 INTERFACE PORT, J6 JTAG, J8 Micro_SD_Card_Det_Hirose_DM3AT, J9 IIC RTC, Q1 CSD19505KCS, Q11 CSD19505KCS, Q12 CSD19505KCS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

Commit message: Some missing copper and minor changes
Routing:
- net +5V: track 137.3 -> 137.9 mm
- added copper zone on F.Cu, net Net-(C7-Pad1)
- added copper zone on B.Cu, net Net-(F2-Pad1)
- added copper zone on F.Cu, net Net-(HS1-Pad1)
